File: motherboard.sch (EAGLE design)
At the start: 44 parts, among them J1 PCIE_EDGE, U1 74HCT08D, U2 DAC5574, U3 AZ4558CMTR-G1

Commit message: Update 9-26
Parts:
- removed C12: (no value), resistor:C-EUC1206
- removed D1, D2, D3, D4, D5, D6, D7, D8: BAS16GW, tide_clock:BAS16GW
- removed J1: PCIE_EDGE, tide_clock:PCIE_EDGE
- removed T2, T3, T4, T5, T6, T7, T8: (no value), transistor:-NPN-SOT23-EBC
- removed U2: DAC5574, tide_clock:DAC5574
- removed U3: AZ4558CMTR-G1, tide_clock:AZ4558CMTR-G1
- added B1, B2, B3, B4, B5, B6: PCIE_SOCKET, tide_clock:PCIE_SOCKET
- added C10, C8, C9: 1uF, resistor:C-EUC0805
- added R13, R14, R15, R16, R17, R18, R19, R20: (no value), resistor:R-US_R0805
- added U$1: RPI_SOCKET, tide_clock:RPI_SOCKET
- added U$10, U$14, U$15, U$16, U$20, U$6: UCM1H331MNL1GS, tide_clock:UCM1H331MNL1GS
- added U$11: ATTINY85, tide_clock:ATTINY85
- added U$12: 47uH, tide_clock:SRN8040TA
- added U$13, U$4: BAT54GW, tide_clock:BAT54GW
- added U$17, U$18, U$19: 1935310, tide_clock:1935310
- added U$2: TC78H620FNG, tide_clock:TC78H620FNG
- added U$21: PCA9540BDP, tide_clock:PCA9540BDP
- added U$22, U$23, U$24, U$25, U$26, U$7: 74HC595_QFN, tide_clock:74HC595_QFN
- added U$5: 330uH, tide_clock:SRN8040TA
- added U$8, U$9: BAS16GW, tide_clock:BAS16GW
- C1: value 100U_CAP -> 22nF; device tide_clock:100U_CAP -> resistor:C-EUC0805
- C11, C7: value (none) -> 1uF; device resistor:C-EUC1206 -> resistor:C-EUC0805
- C2: value 100U_CAP -> 220nF; device tide_clock:100U_CAP -> resistor:C-EUC0805
- C3, C4, C5, C6: value 100U_CAP -> 1uF; device tide_clock:100U_CAP -> resistor:C-EUC0805
- JP1: value JUMPER-SMT_2_NO_SILK_ROUND -> (none); device SparkFun-Jumpers:JUMPER-SMT_2_NO_SILK_ROUND -> pinhead:PINHD-1X3
- JP2: value JUMPER-SMT_2_NO_SILK_ROUND -> (none); device SparkFun-Jumpers:JUMPER-SMT_2_NO_SILK_ROUND -> pinhead:PINHD-1X7
- R10, R3, R4, R5, R6, R7, R8, R9: device resistor:R-US_R1206 -> resistor:R-US_R0805
- R11, R12: device resistor:R-US_R0603 -> resistor:R-US_R0805
- R2: value (none) -> 22k
- U$3: value POWER_EDGE -> TL2575HV-12IKTTR; device tide_clock:POWER_EDGE -> tide_clock:TL2575HV-12IKTTR
- U1: value 74HCT08D -> IFX91041EJV50XUMA1; device tide_clock:74HCT08D -> tide_clock:IFX91041EJV50XUMA1
Connections:
- removed net N$22: T4.B, U2.OUTC
- removed net N$25: R9.2, T3.E
- removed net N$26: R10.2, T4.E
- removed net N$27: R8.1, T6.C
- removed net N$28: R9.1, T7.C
- removed net N$29: R10.1, T8.C
- removed net N$32: JP1.2, R11.1, U2.A0
- removed net N$33: JP2.2, R12.1, U2.A1
- removed net PH_EN1: U1.3A, U1.4A, U3.OUT1
- removed net PH_EN2: U1.1B, U1.2B, U3.OUT2
- removed net SW1: T8.B, U1.1Y
- removed net SW2: T6.B, U1.2Y
- removed net SW3: T5.B, U1.3Y
- removed net SW4: T7.B, U1.4Y
- removed net V+: C6.1, D7.C, D8.C, U$3.A
- new net +12V: U$2.VM, U$3.FB, U$5.2, U$6.1
- new net +3V3: C5.1, U$1.3V3_2, U$2.EN_A, U$2.EN_B, U$2.STBY, U$2.VCC
- new net AT_CS: U$1.10, U$11.PB3
- new net AT_RESET: U$1.3, U$11.RESET
- new net EN10: B3.P2, U$23.Q5
- new net EN11: B3.P3, U$23.Q4
- new net EN12: B3.P6, U$23.Q7
- new net EN13: B4.P1, U$24.Q6
- new net EN14: B4.P2, U$24.Q5
- new net EN15: B4.P3, U$24.Q4
- new net EN16: B4.P6, U$24.Q7
- new net EN17: B5.P1, U$25.Q6
- new net EN18: B5.P2, U$25.Q5
- new net EN19: B5.P3, U$25.Q4
- new net EN20: B5.P6, U$25.Q7
- new net EN21: B6.P1, U$26.Q6
- new net EN22: B6.P2, U$26.Q5
- new net EN23: B6.P3, U$26.Q4
- new net EN24: B6.P6, U$26.Q7
- new net EN5: B2.P1, U$22.Q6
- new net EN6: B2.P2, U$22.Q5
- new net EN7: B2.P3, U$22.Q4
- new net EN8: B2.P6, U$22.Q7
- new net EN9: B3.P1, U$23.Q6
- new net HALL: JP2.7, U$1.21
- new net MISO: U$1.13, U$11.MISO
- new net MOSI: U$1.12, U$11.MOSI
- new net N$14: C6.2, R7.2, U$24.MR
- new net N$15: R18.2, U$22.Q7S, U$23.DS
- new net N$17: C7.2, R8.2, U$23.MR
- new net NEOPIXEL: JP1.3, U$11.PB4
- new net PHA_A: U$1.0, U$2.PHA_A
- new net PHA_B: U$1.2, U$2.PHA_B
- new net SC0: B2.P4, B3.P4, B4.P4, R4.1, U$21.SC0
- new net SC1: B1.P4, B5.P4, B6.P4, R6.1, U$21.SC1
- new net SCK: U$1.14, U$11.SCK
- new net SD0: B2.P5, B3.P5, B4.P5, R3.1, U$21.SD0
- new net SD1: B1.P5, B5.P5, B6.P5, R5.1, U$21.SD1
- new net SDO: R20.2, U$1.15, U$7.DS
- new net SHCP: R13.2, U$1.5, U$22.SHCP, U$23.SHCP, U$24.SHCP, U$25.SHCP, U$26.SHCP, U$7.SHCP
- new net STCP: R14.2, U$1.4, U$22.STCP, U$23.STCP, U$24.STCP, U$25.STCP, U$26.STCP, U$7.STCP
- net +5V: now also B1.5V, B2.5V, B3.5V, B4.5V, B5.5V, B6.5V, C3.2, C4.2, JP2.6, R10.1, R11.1, R12.1, R3.2, R4.2, R5.2, R6.2, R7.1, R8.1, R9.1, U$1.5V, U$1.5V_2, U$11.VCC, U$12.2, U$14.1, U$21.VDD, U$22.VCC, U$23.VCC, U$24.VCC, U$25.VCC, U$26.VCC, U$7.VCC, U1.FB; no longer C11.1, C12.1, C7.1, J1.5V, JP2.1, U1.VCC, U2.VDD, U3.VCC
- net EN1: now also B1.P1, U$7.Q6; no longer J1.P6, U1.4B
- net EN2: now also B1.P2, U$7.Q5; no longer J1.P3, U1.3B
- net EN3: now also B1.P3, U$7.Q4; no longer J1.P2, U1.1A
- net EN4: now also B1.P6, U$7.Q7; no longer J1.P1, U1.2A
- net GND: now also B1.GND, B2.GND, B3.GND, B4.GND, B5.GND, B6.GND, C10.1, C11.1, C3.1, C4.1, C5.2, C6.1, C7.1, C8.1, C9.1, JP1.2, JP2.5, R13.1, R14.1, R15.1, R16.1, R17.1, R18.1, R19.1, R20.1, U$1.GND, U$1.GND_2, U$1.GND_3, U$1.GND_4, U$1.GND_5, U$1.GND_6, U$1.GND_7, U$1.GND_8, U$10.2, U$11.GND, U$13.A, U$14.2, U$15.2, U$16.2, U$18.P$1, U$2.GND, U$20.2, U$21.VSS, U$22.GND, U$22.OE, U$23.GND, U$23.OE, U$24.GND, U$24.OE, U$25.GND, U$25.OE, U$26.GND, U$26.OE, U$3.GND, U$3.ON, U$4.A, U$6.2, U$7.GND, U$7.OE, U1.SYNC; no longer C11.2, C12.2, C3.2, C7.2, D1.A, D2.A, J1.GND, R11.2, R12.2, T5.E, T6.E, T7.E, T8.E, U2.GND, U3.IN1-, U3.IN2+, U3.VEE
- net N$1: now also U1.EN, U1.VS; no longer R7.2
- net N$10: now also JP2.2, U$2.AO2; no longer R4.2, U$3.C2
- net N$11: now also JP2.3, U$2.BO1; no longer R5.2, U$3.C3
- net N$12: now also JP2.4, U$2.BO2; no longer R4.1, T2.C
- net N$13: now also U$3.VOUT, U$4.C, U$5.1; no longer R6.2, U$3.C4
- net N$16: now also R17.2, U$23.Q7S, U$24.DS; no longer R5.1, T3.C
- net N$18: now also C8.2, R9.2, U$22.MR; no longer R6.1, T4.C
- net N$19: now also C9.2, R10.2, U$7.MR; no longer R7.1, T5.C
- net N$2: now also R1.2, T1.B, U$20.1; no longer R1.1, R2.2, U3.IN1+, U3.IN2-
- net N$20: now also R16.2, U$24.Q7S, U$25.DS; no longer T2.B, U2.OUTB
- net N$21: now also C10.2, R11.2, U$25.MR; no longer T3.B, U2.OUTD
- net N$23: now also C11.2, R12.2, U$26.MR; no longer T1.B, U2.OUTA
- net N$24: now also R15.2, U$25.Q7S, U$26.DS; no longer R8.2, T2.E
- net N$3: now also R1.1, U$10.1, U$15.1, U$16.1, U$3.VIN, U$8.C, U$9.C; no longer R3.1
- net N$4: now also C1.2, U1.COMP; no longer C3.1, C6.2, D3.C, D4.C, D5.A, D6.A
- net N$5: now also R2.2; no longer C4.2, D1.C, D3.A
- net N$6: now also C2.2, U1.BDS; no longer C2.1, C5.2, D2.C, D4.A
- net N$7: now also C2.1, U$12.1, U$13.C, U1.BUO; no longer C4.1, D5.C, D7.A
- net N$8: now also R19.2, U$22.DS, U$7.Q7S; no longer C5.1, D6.C, D8.A
- net N$9: now also JP2.1, U$2.AO1; no longer R3.2, U$3.C1
- net PWR1: now also B1.PWR1, B2.PWR1, B3.PWR1, B4.PWR1, B5.PWR1, B6.PWR1, U$17.P$1, U$8.A; no longer C1.2, J1.PWR1, R1.2
- net PWR2: now also B1.PWR2, B2.PWR2, B3.PWR2, B4.PWR2, B5.PWR2, B6.PWR2, U$19.P$1, U$9.A; no longer C2.2, J1.PWR2
- net SCL: now also U$1.9, U$21.SCL; no longer J1.P4, U2.SCL
- net SDA: now also U$1.8, U$21.SDA; no longer J1.P5, U2.SDA
Other:
- moved on the sheet: C1, C11, C2, C3, C4, C5, C6, C7, R1, R10, R11, R12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
